Commit message: Added transmission elements

File: urdf/snake.urdf (robot description, URDF)
Before this commit: robot slither, 21 links, 20 joints
Joints:
- removed joint joint0-1
- removed joint joint1-2
- removed joint joint10-11
- removed joint joint11-12
- removed joint joint12-13
- removed joint joint13-14
- removed joint joint14-15
- removed joint joint15-16
- removed joint joint16-17
- removed joint joint17-18
- removed joint joint18-19
- removed joint joint19-20
- removed joint joint2-3
- removed joint joint3-4
- removed joint joint4-5
- removed joint joint5-6
- removed joint joint6-7
- removed joint joint7-8
- removed joint joint8-9
- removed joint joint9-10
- added joint joint01: type revolute, parent link0, child link1, origin xyz=0 -0.05 0, axis 0 0 1, limit lower=-0.7853981633974483 upper=0.7853981633974483 effort=10.0 velocity=10.0
- added joint joint1011: type revolute, parent link10, child link11, origin xyz=0 -0.1 0, axis 0 0 1, limit lower=-0.7853981633974483 upper=0.7853981633974483 effort=10.0 velocity=10.0
- added joint joint1112: type revolute, parent link11, child link12, origin xyz=0 -0.1 0, axis 0 0 1, limit lower=-0.7853981633974483 upper=0.7853981633974483 effort=10.0 velocity=10.0
- added joint joint12: type revolute, parent link1, child link2, origin xyz=0 -0.1 0, axis 0 0 1, limit lower=-0.7853981633974483 upper=0.7853981633974483 effort=10.0 velocity=10.0
- added joint joint1213: type revolute, parent link12, child link13, origin xyz=0 -0.1 0, axis 0 0 1, limit lower=-0.7853981633974483 upper=0.7853981633974483 effort=10.0 velocity=10.0
- added joint joint1314: type revolute, parent link13, child link14, origin xyz=0 -0.1 0, axis 0 0 1, limit lower=-0.7853981633974483 upper=0.7853981633974483 effort=10.0 velocity=10.0
- added joint joint1415: type revolute, parent link14, child link15, origin xyz=0 -0.1 0, axis 0 0 1, limit lower=-0.7853981633974483 upper=0.7853981633974483 effort=10.0 velocity=10.0
- added joint joint1516: type revolute, parent link15, child link16, origin xyz=0 -0.1 0, axis 0 0 1, limit lower=-0.7853981633974483 upper=0.7853981633974483 effort=10.0 velocity=10.0
- added joint joint1617: type revolute, parent link16, child link17, origin xyz=0 -0.1 0, axis 0 0 1, limit lower=-0.7853981633974483 upper=0.7853981633974483 effort=10.0 velocity=10.0
- added joint joint1718: type revolute, parent link17, child link18, origin xyz=0 -0.1 0, axis 0 0 1, limit lower=-0.7853981633974483 upper=0.7853981633974483 effort=10.0 velocity=10.0
- added joint joint1819: type revolute, parent link18, child link19, origin xyz=0 -0.1 0, axis 0 0 1, limit lower=-0.7853981633974483 upper=0.7853981633974483 effort=10.0 velocity=10.0
- added joint joint1920: type revolute, parent link19, child link20, origin xyz=0 -0.1 0, axis 0 0 1, limit lower=-0.7853981633974483 upper=0.7853981633974483 effort=10.0 velocity=10.0
- added joint joint23: type revolute, parent link2, child link3, origin xyz=0 -0.1 0, axis 0 0 1, limit lower=-0.7853981633974483 upper=0.7853981633974483 effort=10.0 velocity=10.0
- added joint joint34: type revolute, parent link3, child link4, origin xyz=0 -0.1 0, axis 0 0 1, limit lower=-0.7853981633974483 upper=0.7853981633974483 effort=10.0 velocity=10.0
- added joint joint45: type revolute, parent link4, child link5, origin xyz=0 -0.1 0, axis 0 0 1, limit lower=-0.7853981633974483 upper=0.7853981633974483 effort=10.0 velocity=10.0
- added joint joint56: type revolute, parent link5, child link6, origin xyz=0 -0.1 0, axis 0 0 1, limit lower=-0.7853981633974483 upper=0.7853981633974483 effort=10.0 velocity=10.0
- added joint joint67: type revolute, parent link6, child link7, origin xyz=0 -0.1 0, axis 0 0 1, limit lower=-0.7853981633974483 upper=0.7853981633974483 effort=10.0 velocity=10.0
- added joint joint78: type revolute, parent link7, child link8, origin xyz=0 -0.1 0, axis 0 0 1, limit lower=-0.7853981633974483 upper=0.7853981633974483 effort=10.0 velocity=10.0
- added joint joint89: type revolute, parent link8, child link9, origin xyz=0 -0.1 0, axis 0 0 1, limit lower=-0.7853981633974483 upper=0.7853981633974483 effort=10.0 velocity=10.0
- added joint joint910: type revolute, parent link9, child link10, origin xyz=0 -0.1 0, axis 0 0 1, limit lower=-0.7853981633974483 upper=0.7853981633974483 effort=10.0 velocity=10.0
